File: eagle/speakez/mainboard.sch (EAGLE design)
At the start: 22 parts, among them U1 +12v

Commit message: changed clock
Connections:
- net TEST-PINS: now also U$1.D33/PWM/TOUCH; no longer U$1.EXTAL32
Changed lines of the file:
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@@
 <wire x1="30.48" y1="55.88" x2="30.48" y2="45.72" width="0.1524" layer="91"/>
 <junction x="30.48" y="55.88"/>
-<pinref part="U$1" gate="G$1" pin="EXTAL32"/>
-<wire x1="175.26" y1="5.08" x2="180.34" y2="5.08" width="0.1524" layer="91"/>
-<wire x1="180.34" y1="5.08" x2="180.34" y2="-40.64" width="0.1524" layer="91"/>
-<wire x1="180.34" y1="-40.64" x2="73.66" y2="-40.64" width="0.1524" layer="91"/>
-<wire x1="73.66" y1="-40.64" x2="73.66" y2="45.72" width="0.1524" layer="91"/>
+<wire x1="73.66" y1="-17.78" x2="73.66" y2="45.72" width="0.1524" layer="91"/>
 <wire x1="73.66" y1="45.72" x2="30.48" y2="45.72" width="0.1524" layer="91"/>
+<pinref part="U$1" gate="G$1" pin="D33/PWM/TOUCH"/>
+<wire x1="116.84" y1="-17.78" x2="73.66" y2="-17.78" width="0.1524" layer="91"/>
 </segment>
 </net>

Commit message: disconnected battery from V3v3
Connections:
- net N$16: no longer U$1.VOUT3V3
Changed lines of the file:
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@@
 <wire x1="5.08" y1="124.46" x2="5.08" y2="30.48" width="0.1524" layer="91"/>
 <wire x1="144.78" y1="101.6" x2="177.8" y2="101.6" width="0.1524" layer="91"/>
-<wire x1="177.8" y1="101.6" x2="177.8" y2="66.04" width="0.1524" layer="91"/>
+<wire x1="177.8" y1="101.6" x2="177.8" y2="63.5" width="0.1524" layer="91"/>
 <pinref part="U$1" gate="G$1" pin="VCC"/>
-<wire x1="177.8" y1="66.04" x2="177.8" y2="63.5" width="0.1524" layer="91"/>
 <wire x1="177.8" y1="63.5" x2="175.26" y2="63.5" width="0.1524" layer="91"/>
-<pinref part="U$1" gate="G$1" pin="VOUT3V3"/>
-<wire x1="175.26" y1="66.04" x2="177.8" y2="66.04" width="0.1524" layer="91"/>
-<junction x="177.8" y="66.04"/>
 </segment>
 </net>

Commit message: changed clock pin
Connections:
- net TEST-PINS: no longer U$1.D33/PWM/TOUCH
Changed lines of the file:
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@@
 <wire x1="30.48" y1="55.88" x2="30.48" y2="45.72" width="0.1524" layer="91"/>
 <junction x="30.48" y="55.88"/>
-<wire x1="73.66" y1="-17.78" x2="73.66" y2="45.72" width="0.1524" layer="91"/>
-<wire x1="73.66" y1="45.72" x2="30.48" y2="45.72" width="0.1524" layer="91"/>
-<pinref part="U$1" gate="G$1" pin="D33/PWM/TOUCH"/>
-<wire x1="116.84" y1="-17.78" x2="73.66" y2="-17.78" width="0.1524" layer="91"/>
+<wire x1="96.52" y1="45.72" x2="30.48" y2="45.72" width="0.1524" layer="91"/>
+<wire x1="119.38" y1="38.1" x2="96.52" y2="38.1" width="0.1524" layer="91"/>
+<wire x1="96.52" y1="38.1" x2="96.52" y2="45.72" width="0.1524" layer="91"/>
 </segment>
 </net>

Commit message: switched mic in to analog pins
Connections:
- net N$1: now also U$1.D18/A4/SDA0/TOUCH
- net N$2: now also U$1.D19/A5/SCL0/TOUCH
- net N$4: now also U$1.D17/A3/TOUCH; no longer U$1.A12/ADC0_DP3
Changed lines of the file:
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@@
 <wire x1="83.82" y1="38.1" x2="88.9" y2="38.1" width="0.1524" layer="91"/>
 <junction x="83.82" y="38.1"/>
-<wire x1="88.9" y1="38.1" x2="88.9" y2="-27.94" width="0.1524" layer="91"/>
-<wire x1="119.38" y1="-27.94" x2="88.9" y2="-27.94" width="0.1524" layer="91"/>
+<wire x1="88.9" y1="38.1" x2="88.9" y2="20.32" width="0.1524" layer="91"/>
+<pinref part="U$1" gate="G$1" pin="D18/A4/SDA0/TOUCH"/>
+<wire x1="116.84" y1="20.32" x2="88.9" y2="20.32" width="0.1524" layer="91"/>
 </segment>
 </net>
@@
 <pinref part="TESTPINS" gate="A" pin="5"/>
 <wire x1="-12.7" y1="40.64" x2="-20.32" y2="40.64" width="0.1524" layer="91"/>
-<wire x1="86.36" y1="-30.48" x2="86.36" y2="30.48" width="0.1524" layer="91"/>
+<wire x1="86.36" y1="17.78" x2="86.36" y2="30.48" width="0.1524" layer="91"/>
 <wire x1="86.36" y1="30.48" x2="66.04" y2="30.48" width="0.1524" layer="91"/>
 <junction x="66.04" y="30.48"/>
-<wire x1="119.38" y1="-30.48" x2="86.36" y2="-30.48" width="0.1524" layer="91"/>
+<pinref part="U$1" gate="G$1" pin="D19/A5/SCL0/TOUCH"/>
+<wire x1="116.84" y1="17.78" x2="86.36" y2="17.78" width="0.1524" layer="91"/>
 </segment>
 </net>
@@
 <wire x1="-25.4" y1="45.72" x2="-12.7" y2="45.72" width="0.1524" layer="91"/>
 <wire x1="-12.7" y1="45.72" x2="-10.16" y2="45.72" width="0.1524" layer="91"/>
-<wire x1="91.44" y1="-25.4" x2="91.44" y2="40.64" width="0.1524" layer="91"/>
+<wire x1="91.44" y1="22.86" x2="91.44" y2="40.64" width="0.1524" layer="91"/>
 <wire x1="91.44" y1="40.64" x2="48.26" y2="40.64" width="0.1524" layer="91"/>
 <wire x1="48.26" y1="40.64" x2="48.26" y2="30.48" width="0.1524" layer="91"/>
-<pinref part="U$1" gate="G$1" pin="A12/ADC0_DP3"/>
-<wire x1="116.84" y1="-25.4" x2="91.44" y2="-25.4" width="0.1524" layer="91"/>
+<pinref part="U$1" gate="G$1" pin="D17/A3/TOUCH"/>
+<wire x1="116.84" y1="22.86" x2="91.44" y2="22.86" width="0.1524" layer="91"/>
 </segment>
 </net>
@@
 <junction x="43.18" y="73.66"/>
 <wire x1="43.18" y1="73.66" x2="93.98" y2="73.66" width="0.1524" layer="91"/>
-<wire x1="93.98" y1="73.66" x2="93.98" y2="-22.86" width="0.1524" layer="91"/>
-<wire x1="93.98" y1="-22.86" x2="121.92" y2="-22.86" width="0.1524" layer="91"/>
-<wire x1="121.92" y1="-22.86" x2="121.92" y2="-25.4" width="0.1524" layer="91"/>
+<wire x1="93.98" y1="73.66" x2="93.98" y2="25.4" width="0.1524" layer="91"/>
+<wire x1="119.38" y1="25.4" x2="93.98" y2="25.4" width="0.1524" layer="91"/>
 </segment>
 </net>
@@
 </segment>
 </net>
+<net name="N$18" class="0">
+<segment>
+<wire x1="121.92" y1="-22.86" x2="121.92" y2="-25.4" width="0.1524" layer="91"/>
+</segment>
+</net>
